File: dc25badge/dc25badge.kicad_pcb (KiCad board)
At the start: 2 copper layers, 112 parts, among them P1 BATT, P2 USB_OTG, P4 UART, U1 MIC5305, U10 APA102, U11 APA102, U12 APA102, U13 APA102, U14 APA102, U15 APA102, U16 APA102, U17 APA102, U18 APA102, U19 APA102, U2 TPS61232, U20 APA102, U21 APA102, U22 APA102, U23 APA102, U24 APA102, U25 APA102, U26 APA102, U27 APA102, U28 APA102, U29 APA102, U3 ATSAMD21E18A-AU, U30 APA102, U31 APA102, U32 APA102, U33 APA102, U34 APA102, U35 APA102, U36 APA102, U37 APA102, U38 APA102, U39 APA102, U4 74AHCT125, U40 APA102, U41 APA102, U42 APA102, U43 APA102, U44 APA102, U45 APA102, U46 APA102, U47 APA102, U48 APA102, U49 APA102, U5 APA102, U50 APA102, U51 APA102, U52 APA102, U53 APA102, U54 APA102, U55 APA102, U56 APA102, U57 APA102, U58 APA102, U59 APA102, U6 APA102, U60 APA102, U61 APA102, U62 APA102, U63 APA102, U64 APA102, U7 APA102, U8 APA102, U9 APA102, Y1 32.768k

Commit message: Before routing back.
Parts:
- removed BRIGHT: BRIGHT, Buttons_Switches_SMD:SW_SPST_EVQP0
- removed CORTEX: CONN_CORTEX, Pin_Headers2:Pin_Header_Straight_2x05_Pitch1.27mm_SMD
- removed FB1: FB300, Resistors_SMD:R_0805_HandSoldering
- removed MODE: MODE, Buttons_Switches_SMD:SW_SPST_EVQP0
- removed PWR: PWR, Buttons_Switches_SMD:SW_SPST_EVQP0
- removed RESET: RESET, Buttons_Switches_SMD:SW_SPST_EVQP0
- added P3: CONN_CORTEX, Pin_Headers2:Pin_Header_Straight_2x05_Pitch1.27mm_SMD, B.Cu at (86.6, 50.2)
- added SW1: RESET, Buttons_Switches_SMD:SW_SPST_EVQP0, F.Cu at (2.92, 22.5)
- added SW2: PWR, Buttons_Switches_SMD:SW_SPST_EVQP0, F.Cu at (-20.1, 27.8)
- added SW3: MODE, Buttons_Switches_SMD:SW_SPST_EVQP0, F.Cu at (-18.3, 12.4)
- added SW4: BRIGHT, Buttons_Switches_SMD:SW_SPST_EVQP0, F.Cu at (-22.7, -1.27)
- C1, C10, C11, C2, C3, C7, C9, R7, W1, W2, W3: moved to B.Cu
- P2: footprint Connectors:USB_Micro-B -> Badge_Parts:Amphenol_10118192; moved to B.Cu
- moved R5 249.1 mm to (2.29, 31.1)
- moved R6 240.7 mm to (2.54, 41.9)
- moved C8 232.6 mm to (2.54, 36.7)
- moved R7 201.7 mm to (58.5, 37.0)
- moved C7 188.7 mm to (67.4, 45.2), turned to 270 degrees
- moved P2 181.4 mm to (76.7, 31.4)
- moved C3 180.7 mm to (92.5, 32.8), turned to 90 degrees
- moved W2 180.1 mm to (96.3, 29.8)
- moved C9 178.7 mm to (81.9, 38.6), turned to 90 degrees
- moved C10 178.2 mm to (86.5, 38.6), turned to 90 degrees
- moved C11 177.5 mm to (84.2, 38.6), turned to 90 degrees
- moved C2 175.8 mm to (96.3, 38.7)
- moved C1 175.7 mm to (99.9, 32.8), turned to 90 degrees
- moved W1 154.2 mm to (124.3, 33.9)
- moved W3 128.7 mm to (144.5, 51.7)
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Connections:
- C7 pad 1: Net-(C7-Pad1) -> +3V3
- U3 pad 21: BRIGHT -> Net-(U3-Pad21)
- U3 pad 25: MODE -> Net-(U3-Pad25)
- U3 pad 27: SOFT_PWR -> Net-(U3-Pad27)
- U3 pad 6: Net-(U3-Pad6) -> SOFT_PWR
- U3 pad 7: Net-(U3-Pad7) -> MODE
- U3 pad 8: Net-(U3-Pad8) -> BRIGHT
- U3 pad 9: Net-(C7-Pad1) -> +3V3
Routing:
- net GND: track 106.5 -> 112.9 mm, vias 60 -> 59
