File: dc25badge/dc25badge.sch (KiCad schematic (older format))
At the start: 35 parts, among them P1 BATT, P2 USB_OTG, P3 CONN_CORTEX, SW1 RESET, SW2 PWR, SW3 MODE, SW4 BRIGHT, U1 MIC5305, U2 TPS61232, U3 ATSAMD21E18A-AU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

Commit message: Switch to a 48-LED compact design.
Squashed commit of the following:

commit 6f3d96a4927b58100b9ba94752feefb272124e74
Author: David Tomaschik <david@systemoverlord.com>
Date:   Thu Jun 1 00:38:57 2017 -0700

    Update notes.

commit 8834e21676bcc6d408b77b676d72b46c0c38b607
Author: David Tomaschik <david@systemoverlord.com>
Date:   Thu Jun 1 00:36:52 2017 -0700

    Adjust soldermask pullback.

commit 6a323dcd490a4f291170055eb47e88aea6817de8
Author: David Tomaschik <david@systemoverlord.com>
Date:   Thu Jun 1 00:27:20 2017 -0700

    Update gerbers.

commit 7bd1ee053eeeac802e043e2ae021bc15df15862e
Author: David Tomaschik <david@systemoverlord.com>
Date:   Wed May 31 23:57:27 2017 -0700

    Silkscreen fixes.

commit dfae645180f2571b52ff98df1726defa7603401b
Author: David Tomaschik <david@systemoverlord.com>
Date:   Wed May 31 23:53:39 2017 -0700

    Remove NPTH.

commit a8849ea9e6f9fd616038fcef49a894d8de34ea94
Author: David Tomaschik <david@systemoverlord.com>
Date:   Wed May 31 23:52:01 2017 -0700

    48 LED build passes DRC.

commit 7ea769f8f5de26af904e5fc144a52ab725d91849
Author: David Tomaschik <david@systemoverlord.com>
Date:   Wed May 31 23:47:17 2017 -0700

    48 LED rebuild.

commit cfd035b7e2ebecbba1f16bb6ecda1aa97673773e
Author: David Tomaschik <david@systemoverlord.com>
Date:   Wed May 31 15:54:34 2017 -0700

    WIP

commit 41f0ca9e7d168e9e42c8a1df9409238d850c65f5
Author: David Tomaschik <david@systemoverlord.com>
Date:   Wed May 31 11:45:54 2017 -0700

    New board outline, graphics, and LED positions.

commit ffe1b2e410b22eb856250e8cd03ac130fafff124
Author: David Tomaschik <david@systemoverlord.com>
Date:   Wed May 31 09:44:54 2017 -0700

    Schematic changes for 48 LED version.
Parts:
- removed R1: 10k, Resistors_SMD:R_0805_HandSoldering, symbol R_Small
- removed SW2: PWR, Buttons_Switches_SMD:SW_SPST_EVQP0, symbol SW_Push
- C12, C13: footprint Capacitors_SMD:C_0805_HandSoldering -> Capacitors_SMD:C_0603_HandSoldering
- P2: symbol USB_OTG -> USB_OTG-RESCUE-dc25badge
- P3: value CONN_CORTEX -> CORTEX
Connections:
- net MOSI3: now also U4.2 (D); no longer U4.5 (D)
- net SCLK3: now also U3.20 (PA19), U4.5 (D); no longer U3.18 (PA17), U4.2 (D)
- net SPI_CLK: now also U4.6 (O); no longer U4.3 (O)
- net SPI_EN: now also U4.1 (E), U4.4 (E); no longer U4.1 (E), U4.4 (E)
- net SPI_MOSI: now also U4.3 (O); no longer U4.6 (O)
- net VBAT: now also U2.9 (EN)
- net 5V_EN: no longer names the net of U3.25 (PA27)
- net 5V_EN: no longer U2.9 (EN)
- net SOFT_PWR: no longer names the net of U3.6 (PA05)
- no-connect marks 24 -> 26
Changed lines of the file:
@@
 EESchema Schematic File Version 2
+LIBS:dc25badge-rescue
 LIBS:power
 LIBS:device
@@
 	1    0    0    -1
 $EndComp
-Text GLabel 3250 1850 0    60   Input ~ 0
-5V_EN
 Text GLabel 3650 5250 2    60   Input ~ 0
 ~RESET
@@
 P 3000 6800
 F 0 "P3" H 3000 7100 50  0000 C CNN
-F 1 "CONN_CORTEX" H 3000 6500 50  0000 C CNN
+F 1 "CORTEX" H 3000 6500 50  0000 C CNN
 F 2 "Pin_Headers2:Pin_Header_Straight_2x05_Pitch1.27mm_SMD" H 3000 5600 50  0001 C CNN
 F 3 "" H 3000 5600 50  0000 C CNN
@@
 USBD+
 $Comp
-L USB_OTG P2
+L USB_OTG-RESCUE-dc25badge P2
 U 1 1 592AA55B
 P 950 3950
@@
 $Comp
 L 74AHCT125 U4
-U 1 1 592AAF69
+U 2 1 592AAF69
 P 6750 4600
 F 0 "U4" H 6750 4700 50  0000 L BNN
@@
 F 2 "SMD_Packages:SOIC-14_N" H 6750 4600 50  0001 C CNN
 F 3 "" H 6750 4600 50  0000 C CNN
-	1    6750 4600
+	2    6750 4600
 	1    0    0    -1
 $EndComp
 $Comp
 L 74AHCT125 U4
-U 2 1 592AB1CD
+U 1 1 592AB1CD
 P 6750 5100
 F 0 "U4" H 6750 5200 50  0000 L BNN
@@
 F 2 "SMD_Packages:SOIC-14_N" H 6750 5100 50  0001 C CNN
 F 3 "" H 6750 5100 50  0000 C CNN
-	2    6750 5100
+	1    6750 5100
 	1    0    0    -1
 $EndComp
@@
 Text GLabel 7200 5100 2    60   Output ~ 0
 SPI_MOSI
-NoConn ~ 3650 4750
 $Comp
 L R_Small R7
@@
 $EndComp
 $Comp
-L PWR_FLAG #FLG016
-U 1 1 592ACB04
-P 5300 850
-F 0 "#FLG016" H 5300 945 50  0001 C CNN
-F 1 "PWR_FLAG" H 5300 1030 50  0000 C CNN
-F 2 "" H 5300 850 50  0000 C CNN
-F 3 "" H 5300 850 50  0000 C CNN
-	1    5300 850
-	1    0    0    -1
-$EndComp
-$Comp
-L GND #PWR017
+L GND #PWR016
 U 1 1 592ACB78
-P 5300 1000
-F 0 "#PWR017" H 5300 750 50  0001 C CNN
-F 1 "GND" H 5300 850 50  0000 C CNN
-F 2 "" H 5300 1000 50  0000 C CNN
-F 3 "" H 5300 1000 50  0000 C CNN
-	1    5300 1000
+P 5550 950
+F 0 "#PWR016" H 5550 700 50  0001 C CNN
+F 1 "GND" H 5550 800 50  0000 C CNN
+F 2 "" H 5550 950 50  0000 C CNN
+F 3 "" H 5550 950 50  0000 C CNN
+	1    5550 950
 	1    0    0    -1
 $EndComp
@@
 Wire Wire Line
 	7850 4850 7850 4950
-Wire Wire Line
-	5300 850  5300 1000
-Wire Wire Line
-	5550 900  5300 900
-Connection ~ 5300 900
 $Comp
 L 74AHCT125 U4
@@
 $EndComp
 $Comp
-L PWR_FLAG #FLG018
-U 1 1 592AD7E8
-P 2150 850
-F 0 "#FLG018" H 2150 945 50  0001 C CNN
-F 1 "PWR_FLAG" H 2150 1030 50  0000 C CNN
-F 2 "" H 2150 850 50  0000 C CNN
-F 3 "" H 2150 850 50  0000 C CNN
-	1    2150 850
-	1    0    0    -1
-$EndComp
-$Comp
-L PWR_FLAG #FLG019
+L PWR_FLAG #FLG017
 U 1 1 592AD95C
 P 1150 1750
-F 0 "#FLG019" H 1150 1845 50  0001 C CNN
+F 0 "#FLG017" H 1150 1845 50  0001 C CNN
 F 1 "PWR_FLAG" H 1150 1930 50  0000 C CNN
 F 2 "" H 1150 1750 50  0000 C CNN
@@
 	4700 6700 4700 6800
 $Comp
-L +5V #PWR020
+L +5V #PWR018
 U 1 1 592AE3BE
 P 5250 6750
-F 0 "#PWR020" H 5250 6600 50  0001 C CNN
+F 0 "#PWR018" H 5250 6600 50  0001 C CNN
 F 1 "+5V" H 5250 6890 50  0000 C CNN
 F 2 "" H 5250 6750 50  0000 C CNN
@@
 	4250 6400 4250 7200
 $Comp
-L GND #PWR021
+L GND #PWR019
 U 1 1 592AE5B3
 P 4250 7200
-F 0 "#PWR021" H 4250 6950 50  0001 C CNN
+F 0 "#PWR019" H 4250 6950 50  0001 C CNN
 F 1 "GND" H 4250 7050 50  0000 C CNN
 F 2 "" H 4250 7200 50  0000 C CNN
@@
 $EndComp
 Connection ~ 4250 7100
-$Comp
-L PWR_FLAG #FLG022
-U 1 1 592AECA7
-P 1600 5350
-F 0 "#FLG022" H 1600 5445 50  0001 C CNN
-F 1 "PWR_FLAG" H 1600 5530 50  0000 C CNN
-F 2 "" H 1600 5350 50  0000 C CNN
-F 3 "" H 1600 5350 50  0000 C CNN
-	1    1600 5350
-	1    0    0    -1
-$EndComp
 Text GLabel 2200 4750 0    60   Output ~ 0
 TXD
@@
 	2300 4850 2200 4850
 NoConn ~ 3650 4550
-Text GLabel 3750 4250 2    60   Output ~ 0
-5V_EN
-$Comp
-L GND #PWR023
+$Comp
+L GND #PWR020
 U 1 1 592B0060
 P 1350 3500
-F 0 "#PWR023" H 1350 3250 50  0001 C CNN
+F 0 "#PWR020" H 1350 3250 50  0001 C CNN
 F 1 "GND" H 1350 3350 50  0000 C CNN
 F 2 "" H 1350 3500 50  0000 C CNN
@@
 F 0 "C13" H 2560 3470 50  0000 L CNN
 F 1 "22pF" H 2560 3320 50  0000 L CNN
-F 2 "Capacitors_SMD:C_0805_HandSoldering" H 2550 3400 50  0001 C CNN
+F 2 "Capacitors_SMD:C_0603_HandSoldering" H 2550 3400 50  0001 C CNN
 F 3 "" H 2550 3400 50  0000 C CNN
 	1    2550 3400
@@
 F 0 "C12" H 2160 3470 50  0000 L CNN
 F 1 "22pF" H 2160 3320 50  0000 L CNN
-F 2 "Capacitors_SMD:C_0805_HandSoldering" H 2150 3400 50  0001 C CNN
+F 2 "Capacitors_SMD:C_0603_HandSoldering" H 2150 3400 50  0001 C CNN
 F 3 "" H 2150 3400 50  0000 C CNN
 	1    2150 3400
@@
 Connection ~ 2150 3250
 $Comp
-L GND #PWR024
+L GND #PWR021
 U 1 1 592B1083
 P 2350 3600
-F 0 "#PWR024" H 2350 3350 50  0001 C CNN
+F 0 "#PWR021" H 2350 3350 50  0001 C CNN
 F 1 "GND" H 2350 3450 50  0000 C CNN
 F 2 "" H 2350 3600 50  0000 C CNN
@@
 Wire Wire Line
 	2200 4050 2300 4050
-Connection ~ 1600 5350
 Connection ~ 1150 1750
 Text Notes 3850 3200 0    120  ~ 0
@@
 NoConn ~ 2300 4950
 NoConn ~ 2300 5050
-Text GLabel 2200 4450 0    60   Input ~ 0
-SOFT_PWR
 Text GLabel 2200 4550 0    60   Input ~ 0
 MODE
-$Comp
-L SW_Push SW2
-U 1 1 592B9D49
-P 6000 3300
-F 0 "SW2" H 6050 3400 50  0000 L CNN
-F 1 "PWR" H 6000 3240 50  0000 C CNN
-F 2 "Buttons_Switches_SMD:SW_SPST_EVQP0" H 6000 3500 50  0001 C CNN
-F 3 "" H 6000 3500 50  0000 C CNN
-	1    6000 3300
-	1    0    0    -1
-$EndComp
 $Comp
 L SW_Push SW3
@@
 Text GLabel 5700 3550 0    60   Output ~ 0
 MODE
-Text GLabel 5700 3300 0    60   Output ~ 0
-SOFT_PWR
-Wire Wire Line
-	5700 3300 5800 3300
 Wire Wire Line
 	5700 3550 5800 3550
 $Comp
-L GND #PWR025
+L GND #PWR022
 U 1 1 592BA362
 P 6300 3900
-F 0 "#PWR025" H 6300 3650 50  0001 C CNN
+F 0 "#PWR022" H 6300 3650 50  0001 C CNN
 F 1 "GND" H 6300 3750 50  0000 C CNN
 F 2 "" H 6300 3900 50  0000 C CNN
@@
 Wire Wire Line
 	6200 3550 6300 3550
-Wire Wire Line
-	6300 3300 6300 3900
-Wire Wire Line
-	6200 3300 6300 3300
 Connection ~ 6300 3550
 Text GLabel 3750 5050 2    60   Output ~ 0
 MOSI3
-Text GLabel 3750 4950 2    60   Output ~ 0
+Text GLabel 3750 4750 2    60   Output ~ 0
 SCLK3
 Text GLabel 3750 4850 2    60   Output ~ 0
@@
 Wire Wire Line
 	3750 4850 3650 4850
-Wire Wire Line
-	3750 4950 3650 4950
 Wire Wire Line
 	3750 5050 3650 5050
@@
 $EndComp
 $Comp
-L GND #PWR026
+L GND #PWR023
 U 1 1 592C536E
 P 4150 2600
-F 0 "#PWR026" H 4150 2350 50  0001 C CNN
+F 0 "#PWR023" H 4150 2350 50  0001 C CNN
 F 1 "GND" H 4150 2450 50  0000 C CNN
 F 2 "" H 4150 2600 50  0000 C CNN
@@
 	4000 1400 3600 1400
 Wire Wire Line
-	3600 1400 3600 1750
+	3600 1400 3600 1850
 Connection ~ 3600 1750
-$Comp
-L R_Small R1
-U 1 1 592C5F86
-P 3300 2300
-F 0 "R1" H 3330 2320 50  0000 L CNN
-F 1 "10k" H 3330 2260 50  0000 L CNN
-F 2 "Resistors_SMD:R_0805_HandSoldering" H 3300 2300 50  0001 C CNN
-F 3 "" H 3300 2300 50  0000 C CNN
-	1    3300 2300
-	1    0    0    -1
-$EndComp
-Wire Wire Line
-	3300 2200 3300 1850
-Connection ~ 3300 1850
-Wire Wire Line
-	3300 2400 3300 2550
 Connection ~ 3600 2550
 NoConn ~ 3700 1950
 $Comp
-L +5V #PWR027
+L +5V #PWR024
 U 1 1 592C61C0
 P 3500 2050
-F 0 "#PWR027" H 3500 1900 50  0001 C CNN
+F 0 "#PWR024" H 3500 1900 50  0001 C CNN
 F 1 "+5V" H 3500 2190 50  0000 C CNN
 F 2 "" H 3500 2050 50  0000 C CNN
@@
 Connection ~ 2850 1750
 Wire Wire Line
-	3250 1850 3700 1850
-Wire Wire Line
 	2850 2400 2850 2550
-Connection ~ 3300 2550
 $Comp
 L C_Small C6
@@
 NoConn ~ 3650 4650
 Wire Wire Line
-	2200 4450 2300 4450
-Wire Wire Line
 	2300 4550 2200 4550
 Wire Wire Line
@@
 NoConn ~ 1050 3300
 $Comp
-L GND #PWR028
+L GND #PWR025
 U 1 1 592CB85E
 P 850 4400
-F 0 "#PWR028" H 850 4150 50  0001 C CNN
+F 0 "#PWR025" H 850 4150 50  0001 C CNN
 F 1 "GND" H 850 4250 50  0000 C CNN
 F 2 "" H 850 4400 50  0000 C CNN
@@
 Wire Wire Line
 	850  4400 850  4350
+Wire Wire Line
+	5550 900  5550 950
+NoConn ~ 3650 4250
+Wire Wire Line
+	3750 4750 3650 4750
+NoConn ~ 3650 4950
+Wire Wire Line
+	3600 1850 3700 1850
 NoConn ~ 2300 4350
 Wire Wire Line
-	3750 4250 3650 4250
+	6300 3550 6300 3900
+NoConn ~ 2300 4450
 $EndSCHEMATC
