File: protospin/protospin.kicad_pcb (KiCad board)
At the start: 2 copper layers, 35 parts, among them P1 BATT, P2 USB_OTG, P3 CONN_CORTEX, P4 CONN_01X16, SW1 RESET, U1 MIC5305, U2 ATSAMD21E18A-AU, U3 TPS61232, U4 74AHCT125, U5 APA102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

Commit message: Rev A protospin.
Parts:
- removed W1: 3v3, Measurement_Points:Measurement_Point_Round-SMD-Pad_Big
- removed W2: 5v, Measurement_Points:Measurement_Point_Round-SMD-Pad_Big
- removed W3: GND, Measurement_Points:Measurement_Point_Round-SMD-Pad_Big
- P4: footprint Pin_Headers2:Pin_Header_Straight_1x16_Pitch2.54mm_SMD_Pin1Left -> Pin_Headers2:Pin_Header_Straight_1x16_Pitch2.54mm_SMD_Pin1Right
- moved R4 24.0 mm to (134.5, 78.9), turned to 270 degrees
- moved L1 8.19 mm to (165.5, 83.9)
- moved U3 8.19 mm to (165.5, 88.5)
- moved R3 8.19 mm to (167.5, 94.1)
- moved C13 8.19 mm to (157.7, 90.4)
- moved C14 8.19 mm to (162.2, 90.4)
- moved C15 8.19 mm to (159.9, 90.4)
- moved C8 8.19 mm to (170.6, 87.8)
- moved C9 8.19 mm to (167.5, 91.7)
- moved R1 5.39 mm to (129.4, 104.0), turned to 90 degrees
- moved U5 4.06 mm to (158.0, 99.3)
- moved U6 4.06 mm to (164.6, 99.2)
- moved U4 3.75 mm to (150.1, 92.7)
- moved P3 3.32 mm to (121.4, 96.4)
- moved R2 2.79 mm to (121.5, 105.5), turned to 0 degrees
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Connections:
- P1 pad 1: GND -> /VBAT
- P1 pad 2: /VBAT -> GND
- P4 pad 5: SOFT_PWR -> BRIGHT
- P4 pad 7: BRIGHT -> SOFT_PWR
- P4 pad 8: SWDIO -> SWCLK
- P4 pad 9: SWCLK -> SWDIO
Routing:
- net GND: track 0.00 -> 113.8 mm, vias 0 -> 23
- net +3V3: track 0.00 -> 100.6 mm
- net 5V_EN: track 0.00 -> 92.5 mm, vias 0 -> 2
- net +5V: track 0.00 -> 64.2 mm, vias 0 -> 2
- net SWCLK: track 0.00 -> 62.2 mm
- net ~RESET: track 0.00 -> 61.9 mm, vias 0 -> 2
- net /VBAT: track 0.00 -> 55.4 mm
- net SWDIO: track 0.00 -> 45.6 mm
- net BRIGHT: track 0.00 -> 40.3 mm, vias 0 -> 2
- net SOFT_PWR: track 0.00 -> 36.2 mm, vias 0 -> 2
- net MODE: track 0.00 -> 35.0 mm, vias 0 -> 2
- net Net-(P4-Pad4): track 0.00 -> 30.4 mm
- net SPI_EN: track 0.00 -> 28.5 mm, vias 0 -> 3
- net TXD: track 0.00 -> 28.0 mm, vias 0 -> 2
- net RXD: track 0.00 -> 25.4 mm, vias 0 -> 2
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- added copper zone on F.Cu, net +5V
- added copper zone on B.Cu, net GND
- added copper zone on F.Cu, net Net-(L1-Pad2)
Other:
- board outline added: 57.3 x 38.1 mm
- net class Default: clearance 0.2 -> 0.1524; trace_width 0.25 -> 0.1524; via_dia 0.6 -> 0.381; via_drill 0.4 -> 0.254
- rule trace_clearance: 0.2 -> 0.1524
- board text added: "+"
- board text added: "XXV Rev A"
