File: protospin/protospin.sch (KiCad schematic (older format))
At the start: 35 parts, among them P1 BATT, P2 USB_OTG, P3 CONN_CORTEX, SW1 RESET, U1 MIC5305, U2 ATSAMD21E18A-AU, U3 TPS61232, U4 74AHCT125, U5 APA102, U6 APA102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

Commit message: Rev A protospin.
Parts:
- removed W1: 3v3, Measurement_Points:Measurement_Point_Round-SMD-Pad_Big, symbol TEST_1P
- removed W2: 5v, Measurement_Points:Measurement_Point_Round-SMD-Pad_Big, symbol TEST_1P
- removed W3: GND, Measurement_Points:Measurement_Point_Round-SMD-Pad_Big, symbol TEST_1P
- P4: renamed from P?; footprint (none) -> Pin_Headers2:Pin_Header_Straight_1x16_Pitch2.54mm_SMD_Pin1Right
Connections:
- net BRIGHT: now also P4.5 (P5); no longer P4.7 (P7)
- net GND: now also P1.2 (P2); no longer P1.1 (P1)
- net SOFT_PWR: now also P4.7 (P7); no longer P4.5 (P5)
- net SWCLK: now also P4.8 (P8); no longer P4.9 (P9)
- net SWDIO: now also P4.9 (P9); no longer P4.8 (P8)
- net VBAT: now also P1.1 (P1); no longer P1.2 (P2)
Changed lines of the file:
@@
 LIBS:valves
 LIBS:dc25badge
-LIBS:dc25badge-cache
+LIBS:protospin-cache
 EELAYER 25 0
 EELAYER END
@@
 F 3 "" H 800 2500 50  0000 C CNN
 	1    800  2500
-	-1   0    0    1
+	-1   0    0    -1
 $EndComp
 $Comp
@@
 	1    0    0    -1
 $EndComp
-$Comp
-L TEST_1P W1
-U 1 1 592CEE3A
-P 2750 900
-F 0 "W1" H 2750 1170 50  0000 C CNN
-F 1 "3v3" H 2750 1100 50  0000 C CNN
-F 2 "Measurement_Points:Measurement_Point_Round-SMD-Pad_Big" H 2950 900 50  0001 C CNN
-F 3 "" H 2950 900 50  0000 C CNN
-	1    2750 900
-	1    0    0    -1
-$EndComp
-$Comp
-L TEST_1P W2
-U 1 1 592CEE41
-P 5450 2000
-F 0 "W2" H 5450 2270 50  0000 C CNN
-F 1 "5v" H 5450 2200 50  0000 C CNN
-F 2 "Measurement_Points:Measurement_Point_Round-SMD-Pad_Big" H 5650 2000 50  0001 C CNN
-F 3 "" H 5650 2000 50  0000 C CNN
-	1    5450 2000
-	1    0    0    -1
-$EndComp
-$Comp
-L TEST_1P W3
-U 1 1 592CEE48
-P 5600 950
-F 0 "W3" H 5600 1220 50  0000 C CNN
-F 1 "GND" H 5600 1150 50  0000 C CNN
-F 2 "Measurement_Points:Measurement_Point_Round-SMD-Pad_Big" H 5800 950 50  0001 C CNN
-F 3 "" H 5800 950 50  0000 C CNN
-	1    5600 950
-	1    0    0    -1
-$EndComp
 Text GLabel 7250 4650 2    60   Output ~ 0
 SPI_CLK
@@
 Wire Wire Line
 	2450 1000 2450 900
-Wire Wire Line
-	2200 900  2750 900
 Connection ~ 2450 900
 Wire Wire Line
@@
 Wire Wire Line
 	5350 900  5350 1050
-Wire Wire Line
-	5600 950  5350 950
 Connection ~ 5350 950
 $Comp
@@
 Connection ~ 2200 3300
 $Comp
-L GND #PWR024
+L GND #PWR023
 U 1 1 592CEF0E
 P 2400 3650
-F 0 "#PWR024" H 2400 3400 50  0001 C CNN
+F 0 "#PWR023" H 2400 3400 50  0001 C CNN
 F 1 "GND" H 2400 3500 50  0000 C CNN
 F 2 "" H 2400 3650 50  0000 C CNN
@@
 Text GLabel 9150 3950 0    60   Output ~ 0
 MODE
-Text GLabel 9150 3850 0    60   Output ~ 0
+Text GLabel 9150 4050 0    60   Output ~ 0
 SOFT_PWR
 Text GLabel 3800 5100 2    60   Output ~ 0
@@
 Wire Wire Line
 	3700 4500 3800 4500
-Text GLabel 9150 4050 0    60   Output ~ 0
+Text GLabel 9150 3850 0    60   Output ~ 0
 BRIGHT
 Wire Wire Line
@@
 $EndComp
 $Comp
-L GND #PWR025
+L GND #PWR024
 U 1 1 592CEF6A
 P 4200 2650
-F 0 "#PWR025" H 4200 2400 50  0001 C CNN
+F 0 "#PWR024" H 4200 2400 50  0001 C CNN
 F 1 "GND" H 4200 2500 50  0000 C CNN
 F 2 "" H 4200 2650 50  0000 C CNN
@@
 NoConn ~ 3750 2000
 $Comp
-L +5V #PWR026
+L +5V #PWR025
 U 1 1 592CEF99
 P 3550 2100
-F 0 "#PWR026" H 3550 1950 50  0001 C CNN
+F 0 "#PWR025" H 3550 1950 50  0001 C CNN
 F 1 "+5V" H 3550 2240 50  0000 C CNN
 F 2 "" H 3550 2100 50  0000 C CNN
@@
 	2350 4700 2250 4700
 $Comp
-L GND #PWR027
+L GND #PWR026
 U 1 1 592CEFD9
 P 900 4450
-F 0 "#PWR027" H 900 4200 50  0001 C CNN
+F 0 "#PWR026" H 900 4200 50  0001 C CNN
 F 1 "GND" H 900 4300 50  0000 C CNN
 F 2 "" H 900 4450 50  0000 C CNN
@@
 	7300 3500 7250 3500
 $Comp
-L +5V #PWR?
+L +5V #PWR027
 U 1 1 592D0EE8
 P 9100 2800
-F 0 "#PWR?" H 9100 2650 50  0001 C CNN
+F 0 "#PWR027" H 9100 2650 50  0001 C CNN
 F 1 "+5V" H 9100 2940 50  0000 C CNN
 F 2 "" H 9100 2800 50  0000 C CNN
@@
 $EndComp
 $Comp
-L +3V3 #PWR?
+L +3V3 #PWR028
 U 1 1 592D0F46
 P 9100 3000
-F 0 "#PWR?" H 9100 2850 50  0001 C CNN
+F 0 "#PWR028" H 9100 2850 50  0001 C CNN
 F 1 "+3V3" H 9100 3140 50  0000 C CNN
 F 2 "" H 9100 3000 50  0000 C CNN
@@
 $EndComp
 $Comp
-L GND #PWR?
+L GND #PWR029
 U 1 1 592D0FA4
 P 9150 4700
-F 0 "#PWR?" H 9150 4450 50  0001 C CNN
+F 0 "#PWR029" H 9150 4450 50  0001 C CNN
 F 1 "GND" H 9150 4550 50  0000 C CNN
 F 2 "" H 9150 4700 50  0000 C CNN
@@
 	1    0    0    -1
 $EndComp
-Text GLabel 9150 4150 0    60   BiDi ~ 0
+Text GLabel 9150 4250 0    60   BiDi ~ 0
 SWDIO
-Text GLabel 9150 4250 0    60   Output ~ 0
+Text GLabel 9150 4150 0    60   Output ~ 0
 SWCLK
 Text GLabel 9150 4350 0    60   Output ~ 0
@@
 RXD
 $Comp
-L CONN_01X16 P?
+L CONN_01X16 P4
 U 1 1 592D1E73
 P 9900 3950
-F 0 "P?" H 9900 4800 50  0000 C CNN
+F 0 "P4" H 9900 4800 50  0000 C CNN
 F 1 "CONN_01X16" V 10000 3950 50  0000 C CNN
-F 2 "" H 9900 3950 50  0000 C CNN
+F 2 "Pin_Headers2:Pin_Header_Straight_1x16_Pitch2.54mm_SMD_Pin1Right" H 9900 3950 50  0001 C CNN
 F 3 "" H 9900 3950 50  0000 C CNN
 	1    9900 3950
@@
 Connection ~ 9700 4600
 Connection ~ 9700 4500
+Wire Wire Line
+	2450 900  2200 900
 $EndSCHEMATC

Commit message: Protospin stuff.
Parts:
- U1: symbol MIC5305 -> MIC5305-RESCUE-protospin
Changed lines of the file:
@@
 EESchema Schematic File Version 2
+LIBS:protospin-rescue
 LIBS:power
 LIBS:device
@@
 $EndComp
 $Comp
-L MIC5305 U1
+L MIC5305-RESCUE-protospin U1
 U 1 1 592CED5B
 P 1700 1600
